File: Shakey.sch (EAGLE design)
At the start: 81 parts, among them CN1 CONN_USB-4UCON-11071, CN2 ISP, U1 ATMEGA32U4-AU, U2 ICM-20689, U3 AP2210K-3.3TRG1, U4 LM75AD, Y1 16Mhz

Commit message: completed
Parts:
- renumbered CN2 to ISP, LED7 to TX_LED, LED8 to RX_LED, LED9 to ON
Changed lines of the file:
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@@
 <part name="R12" library="rcl" deviceset="R-EU_" device="R0603" value="330R"/>
 <part name="P+4" library="supply1" deviceset="VCC" device=""/>
-<part name="CN2" library="SixthLogic" deviceset="DEBUGPORT-6PIN" device="-ISP-AVR" value="ISP"/>
+<part name="ISP" library="SixthLogic" deviceset="DEBUGPORT-6PIN" device="-ISP-AVR" value="ISP"/>
 <part name="P+5" library="supply1" deviceset="VCC" device=""/>
 <part name="SUPPLY8" library="supply2" deviceset="GND" device=""/>
@@
 <part name="P+7" library="supply1" deviceset="VCC" device=""/>
 <part name="SJ1" library="SixthLogic" deviceset="SOLDER_JUMPER_NC" device="" value="SOLDER JUMPER"/>
-<part name="LED7" library="SixthLogic" deviceset="LED" device="-1206-LTST-BOTTOM" value="YELLOW"/>
-<part name="LED8" library="SixthLogic" deviceset="LED" device="-1206-LTST-BOTTOM" value="YELLOW"/>
-<part name="LED9" library="SixthLogic" deviceset="LED" device="-1206-LTST-BOTTOM" value="RED"/>
+<part name="TX_LED" library="SixthLogic" deviceset="LED" device="-1206-LTST-BOTTOM" value="YELLOW"/>
+<part name="RX_LED" library="SixthLogic" deviceset="LED" device="-1206-LTST-BOTTOM" value="YELLOW"/>
+<part name="ON" library="SixthLogic" deviceset="LED" device="-1206-LTST-BOTTOM" value="RED"/>
 <part name="R25" library="rcl" deviceset="R-EU_" device="R0603" value="1K"/>
 <part name="R26" library="rcl" deviceset="R-EU_" device="R0603" value="1K"/>
@@
 </instance>
 <instance part="P+4" gate="VCC" x="386.08" y="149.86"/>
-<instance part="CN2" gate="G$1" x="149.86" y="27.94"/>
+<instance part="ISP" gate="G$1" x="149.86" y="27.94"/>
 <instance part="P+5" gate="VCC" x="162.56" y="38.1"/>
 <instance part="SUPPLY8" gate="GND" x="162.56" y="20.32" smashed="yes">
@@
 <attribute name="VALUE" x="106.68" y="52.197" size="1.778" layer="96" rot="R90"/>
 </instance>
-<instance part="LED7" gate="G$1" x="256.54" y="66.04"/>
-<instance part="LED8" gate="G$1" x="266.7" y="66.04"/>
-<instance part="LED9" gate="G$1" x="276.86" y="66.04"/>
+<instance part="TX_LED" gate="G$1" x="256.54" y="66.04"/>
+<instance part="RX_LED" gate="G$1" x="266.7" y="66.04"/>
+<instance part="ON" gate="G$1" x="276.86" y="66.04"/>
 <instance part="R25" gate="G$1" x="256.54" y="76.2" smashed="yes" rot="R90">
 <attribute name="NAME" x="255.0414" y="73.66" size="1.778" layer="95" rot="R90"/>
@@
 </segment>
 <segment>
-<pinref part="CN2" gate="G$1" pin="6"/>
+<pinref part="ISP" gate="G$1" pin="6"/>
 <wire x1="160.02" y1="25.4" x2="162.56" y2="25.4" width="0.1524" layer="91"/>
 <wire x1="162.56" y1="25.4" x2="162.56" y2="22.86" width="0.1524" layer="91"/>
@@
 </segment>
 <segment>
-<pinref part="LED9" gate="G$1" pin="C"/>
+<pinref part="ON" gate="G$1" pin="C"/>
 <pinref part="SUPPLY9" gate="GND" pin="GND"/>
 <wire x1="276.86" y1="60.96" x2="276.86" y2="53.34" width="0.1524" layer="91"/>
@@
 </segment>
 <segment>
-<pinref part="CN2" gate="G$1" pin="2"/>
+<pinref part="ISP" gate="G$1" pin="2"/>
 <wire x1="160.02" y1="30.48" x2="162.56" y2="30.48" width="0.1524" layer="91"/>
 <pinref part="P+5" gate="VCC" pin="VCC"/>
@@
 </segment>
 <segment>
-<pinref part="CN2" gate="G$1" pin="5"/>
+<pinref part="ISP" gate="G$1" pin="5"/>
 <wire x1="139.7" y1="25.4" x2="134.62" y2="25.4" width="0.1524" layer="91"/>
 <label x="134.62" y="25.4" size="1.27" layer="95" rot="R180" xref="yes"/>
@@
 </segment>
 <segment>
-<pinref part="CN2" gate="G$1" pin="3"/>
+<pinref part="ISP" gate="G$1" pin="3"/>
 <wire x1="139.7" y1="27.94" x2="134.62" y2="27.94" width="0.1524" layer="91"/>
 <label x="134.62" y="27.94" size="1.27" layer="95" rot="R180" xref="yes"/>
@@
 </segment>
 <segment>
-<pinref part="CN2" gate="G$1" pin="1"/>
+<pinref part="ISP" gate="G$1" pin="1"/>
 <wire x1="139.7" y1="30.48" x2="134.62" y2="30.48" width="0.1524" layer="91"/>
 <label x="134.62" y="30.48" size="1.27" layer="95" rot="R180" xref="yes"/>
@@
 </segment>
 <segment>
-<pinref part="CN2" gate="G$1" pin="4"/>
+<pinref part="ISP" gate="G$1" pin="4"/>
 <wire x1="160.02" y1="27.94" x2="165.1" y2="27.94" width="0.1524" layer="91"/>
 <label x="165.1" y="27.94" size="1.27" layer="95" xref="yes"/>
@@
 <pinref part="U1" gate="U1" pin="(XCK1/!CTS!)PD5"/>
 <wire x1="177.8" y1="58.42" x2="256.54" y2="58.42" width="0.1524" layer="91"/>
-<pinref part="LED7" gate="G$1" pin="C"/>
+<pinref part="TX_LED" gate="G$1" pin="C"/>
 <wire x1="256.54" y1="58.42" x2="256.54" y2="60.96" width="0.1524" layer="91"/>
 <label x="195.58" y="59.055" size="1.27" layer="95"/>
@@
 <segment>
 <pinref part="U1" gate="U1" pin="(SS/PCINT0)PB0"/>
-<pinref part="LED8" gate="G$1" pin="C"/>
+<pinref part="RX_LED" gate="G$1" pin="C"/>
 <wire x1="177.8" y1="55.88" x2="266.7" y2="55.88" width="0.1524" layer="91"/>
 <wire x1="266.7" y1="55.88" x2="266.7" y2="60.96" width="0.1524" layer="91"/>
@@
 <net name="N$17" class="0">
 <segment>
-<pinref part="LED7" gate="G$1" pin="A"/>
+<pinref part="TX_LED" gate="G$1" pin="A"/>
 <pinref part="R25" gate="G$1" pin="1"/>
 <wire x1="256.54" y1="68.58" x2="256.54" y2="71.12" width="0.1524" layer="91"/>
@@
 <net name="N$18" class="0">
 <segment>
-<pinref part="LED8" gate="G$1" pin="A"/>
+<pinref part="RX_LED" gate="G$1" pin="A"/>
 <pinref part="R26" gate="G$1" pin="1"/>
 <wire x1="266.7" y1="68.58" x2="266.7" y2="71.12" width="0.1524" layer="91"/>
@@
 <net name="N$19" class="0">
 <segment>
-<pinref part="LED9" gate="G$1" pin="A"/>
+<pinref part="ON" gate="G$1" pin="A"/>
 <pinref part="R27" gate="G$1" pin="1"/>
 <wire x1="276.86" y1="68.58" x2="276.86" y2="71.12" width="0.1524" layer="91"/>

Commit message: added BOM with attributes
Parts:
- C1, C2: DESCRIPTION (none) -> CAP CER 22PF 16V C0G/NP0 0603; MF (none) -> KEMET; MPN (none) -> C0603C220K4GACTU; OC_DIGIKEY (none) -> 399-9031-2-ND; SUPPLIER (none) -> Digikey; UNITPRICE (none) -> $0.01675; URL (none) -> https://www.digikey.com/product-detail/en/kemet/C0603C220K4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
- C10, C4, C6: DESCRIPTION (none) -> CAP CER 0.1UF 50V X7R 0603; MF (none) -> Samsung Electro-Mechanics; MPN (none) -> CL10B104KB8NNNC; OC_DIGIKEY (none) -> 1276-1000-2-ND; SUPPLIER (none) -> Digikey; UNITPRICE (none) -> $0.00652; URL (none) -> https://www.digikey.com/product-detail/en/samsung-electro-m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
- C3, C5, C8: DESCRIPTION (none) -> CAP CER 1UF 25V X5R 0603; MF (none) -> Samsung Electro-Mechanics; MPN (none) -> CL10A105KA8NNNC; OC_DIGIKEY (none) -> 1276-1102-2-ND; SUPPLIER (none) -> Digikey; UNITPRICE (none) -> $0.00785; URL (none) -> https://www.digikey.com/product-detail/en/samsung-electro-m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
- C7: DESCRIPTION (none) -> CAP CER 2.2UF 16V X5R 0603; MF (none) -> Samsung Electro-Mechanics; MPN (none) -> CL10A225KO8NNNC; OC_DIGIKEY (none) -> 1276-1040-2-ND; SUPPLIER (none) -> Digikey; UNITPRICE (none) -> $0.01863; URL (none) -> https://www.digikey.com/product-detail/en/samsung-electro-m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
- C9: DESCRIPTION (none) -> CAP CER 0.47UF 16V X7R 0603; MF (none) -> Murata Electronics North America; MPN (none) -> GCM188R71C474KA55D; OC_DIGIKEY (none) -> 490-4775-2-ND; SUPPLIER (none) -> Digikey; UNITPRICE (none) -> $0.03744; URL (none) -> https://www.digikey.com/product-detail/en/murata-electronic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
- F1: DESCRIPTION (none) -> PTC RESET FUSE 8V 500MA 1206; MF (none) -> Bel Fuse Inc.; MPN (none) -> 0ZCJ0050FF2G; OC_DIGIKEY (none) -> 507-1802-6-ND; SUPPLIER (none) -> Digikey; UNITPRICE (none) -> $0.07588; URL (none) -> https://www.digikey.com/product-detail/en/bel-fuse-inc/0ZCJ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
- LED_CLICK, LED_DOWN, LED_LEFT, LED_RIGHT, LED_SPACE, LED_UP: DESCRIPTION (none) -> LED GREEN CLEAR CHIP SMD; MF (none) -> Lite-On Inc.; MPN (none) -> LTST-C230KGKT; OC_DIGIKEY (none) -> 160-1456-2-ND; SUPPLIER (none) -> Digikey; UNITPRICE (none) -> $0.05693; URL (none) -> https://www.digikey.com/product-detail/en/lite-on-inc/LTST-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
- ON: DESCRIPTION (none) -> LED RED CLEAR CHIP SMD; MF (none) -> Lite-On Inc.; MPN (none) -> LTST-C230KRKT; OC_DIGIKEY (none) -> 160-1457-2-ND; SUPPLIER (none) -> Digikey; UNITPRICE (none) -> $0.05668; URL (none) -> https://www.digikey.com/product-detail/en/lite-on-inc/LTST-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
- PC1: DESCRIPTION (none) -> CAP TANT 10UF 20V 10% 2312; MF (none) -> KEMET; MPN (none) -> T491C106K020AT7280; OC_DIGIKEY (none) -> 399-10158-2-ND; SUPPLIER (none) -> Digikey; UNITPRICE (none) -> $0.15113; URL (none) -> https://www.digikey.com/product-detail/en/kemet/T491C106K02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
- R1, R2: DESCRIPTION (none) -> RES 22 OHM 5% 1/10W 0603; MF (none) -> Stackpole Electronics Inc.; MPN (none) -> RMCF0603JT22R0; OC_DIGIKEY (none) -> RMCF0603JT22R0TR-ND; SUPPLIER (none) -> Digikey; UNITPRICE (none) -> $0.00196; URL (none) -> https://www.digikey.com/product-detail/en/stackpole-electro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
- R10, R11, R12: DESCRIPTION (none) -> RES 330 OHM 5% 1/10W 0603; MF (none) -> Stackpole Electronics Inc.; MPN (none) -> RMCF0603JT330R; OC_DIGIKEY (none) -> RMCF0603JT330RTR-ND; SUPPLIER (none) -> Digikey; UNITPRICE (none) -> $0.00196; URL (none) -> https://www.digikey.com/product-detail/en/stackpole-electro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
- R13, R14, R17, R18, R19, R20, R21, R22, R23, R24, R4, R5, R6, R7, R8, R9: DESCRIPTION (none) -> RES SMD 22M OHM 10% 1/10W 0603; MF (none) -> Panasonic Electronic Components; MPN (none) -> ERJ-3GEYK226V; OC_DIGIKEY (none) -> P22MGTR-ND; SUPPLIER (none) -> Digikey; UNITPRICE (none) -> $0.00335; URL (none) -> https://www.digikey.com/product-detail/en/panasonic-electro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
- R25, R26, R27: DESCRIPTION (none) -> RES SMD 1K OHM 5% 1/10W 0603; MF (none) -> Yageo; MPN (none) -> RC0603JR-071KL; OC_DIGIKEY (none) -> 311-1.0KGRTR-ND; SUPPLIER (none) -> Digikey; UNITPRICE (none) -> $0.00268; URL (none) -> https://www.digikey.com/product-detail/en/yageo/RC0603JR-07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
- R28, R29, R3, R30, R31: DESCRIPTION (none) -> RES 10K OHM 5% 1/10W 0603; MF (none) -> Stackpole Electronics Inc.; MPN (none) -> RMCF0603JG10K0; OC_DIGIKEY (none) -> RMCF0603JG10K0TR-ND; SUPPLIER (none) -> Digikey; UNITPRICE (none) -> $0.00170; URL (none) -> https://www.digikey.com/product-detail/en/stackpole-electro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
- RX_LED, TX_LED: DESCRIPTION (none) -> LED YELLOW CLEAR CHIP SMD; MF (none) -> Lite-On Inc.; MPN (none) -> LTST-C230KSKT; OC_DIGIKEY (none) -> 160-1458-2-ND; SUPPLIER (none) -> Digikey; UNITPRICE (none) -> $0.05595; URL (none) -> https://www.digikey.com/product-detail/en/lite-on-inc/LTST-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
- TR1, TR2: DESCRIPTION (none) -> MOSFET N-CH 50V 220MA SOT-23; MF (none) -> ON Semiconductor; MPN (none) -> BSS138; OC_DIGIKEY (none) -> BSS138TR-ND; SUPPLIER (none) -> Digikey; UNITPRICE (none) -> $0.05419; URL (none) -> https://www.digikey.com/product-detail/en/on-semiconductor/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
- U1: UNITPRICE (none) -> $3.04
- U2: DESCRIPTION (none) -> IMU ACCEL/GYRO/TEMP I2C/SPI QFN; MF (none) -> TDK InvenSense; MPN (none) -> ICM-20689; OC_DIGIKEY (none) -> 1428-1059-2-ND; SUPPLIER (none) -> Digikey; UNITPRICE (none) -> $2.62548; URL (none) -> https://www.digikey.com/product-detail/en/tdk-invensense/IC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
- U3: UNITPRICE (none) -> $0.10797
- U4: DESCRIPTION (none) -> SENSOR DIGITAL -55C-125C 8SO; MF (none) -> NXP USA Inc.; MPN (none) -> LM75AD,118; OC_DIGIKEY (none) -> 568-10295-2-ND; SUPPLIER (none) -> Digikey; UNITPRICE (none) -> $0.28743; URL (none) -> https://www.digikey.com/product-detail/en/nxp-usa-inc/LM75A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
- Y1: DESCRIPTION (none) -> CRYSTAL 16.0000MHZ 18PF SMD; MF (none) -> EPSON; MPN (none) -> FA-238 16.0000MB-C3; OC_DIGIKEY (none) -> SER3686TR-ND; SUPPLIER (none) -> Digikey; UNITPRICE (none) -> $0.22880; URL (none) -> https://www.digikey.com/product-detail/en/epson/FA-238-16.0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

Commit message: added fiducial, branding text,logo
Parts:
- added U$7, U$8: FIDUCIAL-1X3MM, SixthLogic:FIDUCIAL-1X3MM
- A, CLICK, DOWN, EARTH1, EARTH2, EARTH3, EARTH4, EARTH5, F, G, LEFT, MOUSE-DOWN, MOUSE-LEFT, MOUSE-LEFT-CLICK, MOUSE-RIGHT, MOUSE-RIGHT-CLICK, MOUSE-UP, RIGHT, SPACE, UP, W: value MA01-1-ALLIGATOR-3MM -> MA01-1-ALLIGATOR-3.1MM; device SixthLogic:MA01-1-ALLIGATOR-3MM -> SixthLogic:MA01-1-ALLIGATOR-3.1MM
Changed lines of the file:
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@@
 <setting verticaltext="up"/>
 </settings>
-<grid distance="0.1" unitdist="inch" unit="inch" style="lines" multiple="1" display="yes" altdistance="0.01" altunitdist="inch" altunit="inch"/>
+<grid distance="0.1" unitdist="inch" unit="inch" style="lines" multiple="1" display="no" altdistance="0.01" altunitdist="inch" altunit="inch"/>
 <layers>
 <layer number="1" name="Top" color="4" fill="1" visible="no" active="no"/>
@@
 <layer number="27" name="tValues" color="7" fill="1" visible="no" active="no"/>
 <layer number="28" name="bValues" color="7" fill="1" visible="no" active="no"/>
-<layer number="29" name="tStop" color="3" fill="3" visible="no" active="no"/>
+<layer number="29" name="tStop" color="7" fill="3" visible="no" active="no"/>
 <layer number="30" name="bStop" color="7" fill="6" visible="no" active="no"/>
-<layer number="31" name="tCream" color="11" fill="1" visible="no" active="no"/>
+<layer number="31" name="tCream" color="10" fill="4" visible="no" active="no"/>
 <layer number="32" name="bCream" color="7" fill="5" visible="no" active="no"/>
 <layer number="33" name="tFinish" color="6" fill="3" visible="no" active="no"/>
@@
 <layer number="37" name="tTest" color="7" fill="1" visible="no" active="no"/>
 <layer number="38" name="bTest" color="7" fill="1" visible="no" active="no"/>
-<layer number="39" name="tKeepout" color="13" fill="1" visible="no" active="no"/>
-<layer number="40" name="bKeepout" color="5" fill="1" visible="no" active="no"/>
+<layer number="39" name="tKeepout" color="4" fill="11" visible="no" active="no"/>
+<layer number="40" name="bKeepout" color="1" fill="11" visible="no" active="no"/>
 <layer number="41" name="tRestrict" color="4" fill="10" visible="no" active="no"/>
 <layer number="42" name="bRestrict" color="1" fill="10" visible="no" active="no"/>
@@
 <layer number="44" name="Drills" color="7" fill="1" visible="no" active="no"/>
 <layer number="45" name="Holes" color="7" fill="1" visible="no" active="no"/>
-<layer number="46" name="Milling" color="12" fill="1" visible="no" active="no"/>
+<layer number="46" name="Milling" color="3" fill="1" visible="no" active="no"/>
 <layer number="47" name="Measures" color="7" fill="1" visible="no" active="no"/>
 <layer number="48" name="Document" color="7" fill="1" visible="no" active="no"/>
@@
 </part>
 <part name="P+3" library="supply1" deviceset="VCC" device=""/>
-<part name="UP" library="SixthLogic" deviceset="MA01-1-ALLIGATOR-3MM" device="" value=""/>
-<part name="LEFT" library="SixthLogic" deviceset="MA01-1-ALLIGATOR-3MM" device="" value=""/>
-<part name="DOWN" library="SixthLogic" deviceset="MA01-1-ALLIGATOR-3MM" device="" value=""/>
-<part name="RIGHT" library="SixthLogic" deviceset="MA01-1-ALLIGATOR-3MM" device="" value=""/>
-<part name="SPACE" library="SixthLogic" deviceset="MA01-1-ALLIGATOR-3MM" device="" value=""/>
-<part name="CLICK" library="SixthLogic" deviceset="MA01-1-ALLIGATOR-3MM" device="" value=""/>
+<part name="UP" library="SixthLogic" deviceset="MA01-1-ALLIGATOR" device="-3.1MM" value=""/>
+<part name="LEFT" library="SixthLogic" deviceset="MA01-1-ALLIGATOR" device="-3.1MM" value=""/>
+<part name="DOWN" library="SixthLogic" deviceset="MA01-1-ALLIGATOR" device="-3.1MM" value=""/>
+<part name="RIGHT" library="SixthLogic" deviceset="MA01-1-ALLIGATOR" device="-3.1MM" value=""/>
+<part name="SPACE" library="SixthLogic" deviceset="MA01-1-ALLIGATOR" device="-3.1MM" value=""/>
+<part name="CLICK" library="SixthLogic" deviceset="MA01-1-ALLIGATOR" device="-3.1MM" value=""/>
 <part name="R4" library="rcl" deviceset="R-EU_" device="R0603" value="22M">
 <attribute name="DESCRIPTION" value="RES SMD 22M OHM 10% 1/10W 0603"/>
@@
 <attribute name="URL" value="https://www.digikey.com/product-detail/en/panasonic-electronic-components/ERJ-3GEYK226V/P22MGTR-ND/282153"/>
 </part>
-<part name="EARTH1" library="SixthLogic" deviceset="MA01-1-ALLIGATOR-3MM" device="" value=""/>
-<part name="EARTH2" library="SixthLogic" deviceset="MA01-1-ALLIGATOR-3MM" device="" value=""/>
-<part name="EARTH3" library="SixthLogic" deviceset="MA01-1-ALLIGATOR-3MM" device="" value=""/>
-<part name="EARTH4" library="SixthLogic" deviceset="MA01-1-ALLIGATOR-3MM" device="" value=""/>
-<part name="EARTH5" library="SixthLogic" deviceset="MA01-1-ALLIGATOR-3MM" device="" value=""/>
+<part name="EARTH1" library="SixthLogic" deviceset="MA01-1-ALLIGATOR" device="-3.1MM" value=""/>
+<part name="EARTH2" library="SixthLogic" deviceset="MA01-1-ALLIGATOR" device="-3.1MM" value=""/>
+<part name="EARTH3" library="SixthLogic" deviceset="MA01-1-ALLIGATOR" device="-3.1MM" value=""/>
+<part name="EARTH4" library="SixthLogic" deviceset="MA01-1-ALLIGATOR" device="-3.1MM" value=""/>
+<part name="EARTH5" library="SixthLogic" deviceset="MA01-1-ALLIGATOR" device="-3.1MM" value=""/>
 <part name="SUPPLY7" library="supply2" deviceset="GND" device=""/>
 <part name="LED_DOWN" library="SixthLogic" deviceset="LED" device="-1206-LTST-BOTTOM" value="GREEN">
@@
 <part name="P+5" library="supply1" deviceset="VCC" device=""/>
 <part name="SUPPLY8" library="supply2" deviceset="GND" device=""/>
-<part name="G" library="SixthLogic" deviceset="MA01-1-ALLIGATOR-3MM" device="" value=""/>
-<part name="F" library="SixthLogic" deviceset="MA01-1-ALLIGATOR-3MM" device="" value=""/>
-<part name="A" library="SixthLogic" deviceset="MA01-1-ALLIGATOR-3MM" device="" value=""/>
-<part name="W" library="SixthLogic" deviceset="MA01-1-ALLIGATOR-3MM" device="" value=""/>
+<part name="G" library="SixthLogic" deviceset="MA01-1-ALLIGATOR" device="-3.1MM" value=""/>
+<part name="F" library="SixthLogic" deviceset="MA01-1-ALLIGATOR" device="-3.1MM" value=""/>
+<part name="A" library="SixthLogic" deviceset="MA01-1-ALLIGATOR" device="-3.1MM" value=""/>
+<part name="W" library="SixthLogic" deviceset="MA01-1-ALLIGATOR" device="-3.1MM" value=""/>
 <part name="R13" library="rcl" deviceset="R-EU_" device="R0603" value="22M">
 <attribute name="DESCRIPTION" value="RES SMD 22M OHM 10% 1/10W 0603"/>
@@
 </part>
 <part name="P+6" library="supply1" deviceset="VCC" device=""/>
-<part name="MOUSE-LEFT-CLICK" library="SixthLogic" deviceset="MA01-1-ALLIGATOR-3MM" device="" value=""/>
-<part name="MOUSE-RIGHT-CLICK" library="SixthLogic" deviceset="MA01-1-ALLIGATOR-3MM" device="" value=""/>
-<part name="MOUSE-RIGHT" library="SixthLogic" deviceset="MA01-1-ALLIGATOR-3MM" device="" value=""/>
-<part name="MOUSE-LEFT" library="SixthLogic" deviceset="MA01-1-ALLIGATOR-3MM" device="" value=""/>
-<part name="MOUSE-DOWN" library="SixthLogic" deviceset="MA01-1-ALLIGATOR-3MM" device="" value=""/>
-<part name="MOUSE-UP" library="SixthLogic" deviceset="MA01-1-ALLIGATOR-3MM" device="" value=""/>
+<part name="MOUSE-LEFT-CLICK" library="SixthLogic" deviceset="MA01-1-ALLIGATOR" device="-3.1MM" value=""/>
+<part name="MOUSE-RIGHT-CLICK" library="SixthLogic" deviceset="MA01-1-ALLIGATOR" device="-3.1MM" value=""/>
+<part name="MOUSE-RIGHT" library="SixthLogic" deviceset="MA01-1-ALLIGATOR" device="-3.1MM" value=""/>
+<part name="MOUSE-LEFT" library="SixthLogic" deviceset="MA01-1-ALLIGATOR" device="-3.1MM" value=""/>
+<part name="MOUSE-DOWN" library="SixthLogic" deviceset="MA01-1-ALLIGATOR" device="-3.1MM" value=""/>
+<part name="MOUSE-UP" library="SixthLogic" deviceset="MA01-1-ALLIGATOR" device="-3.1MM" value=""/>
 <part name="R19" library="rcl" deviceset="R-EU_" device="R0603" value="22M">
 <attribute name="DESCRIPTION" value="RES SMD 22M OHM 10% 1/10W 0603"/>
@@
 <part name="SUPPLY18" library="supply2" deviceset="GND" device=""/>
 <part name="U$6" library="SixthLogic" deviceset="3.3V" device=""/>
+<part name="U$7" library="SixthLogic" deviceset="FIDUCIAL" device="-1X3MM"/>
+<part name="U$8" library="SixthLogic" deviceset="FIDUCIAL" device="-1X3MM"/>
 </parts>
 <sheets>
@@
 </instance>
 <instance part="U$6" gate="G$1" x="287.02" y="256.54"/>
+<instance part="U$7" gate="G$1" x="423.164" y="26.67"/>
+<instance part="U$8" gate="G$1" x="417.83" y="26.67"/>
 </instances>
 <busses>
@@
 <wire x1="375.92" y1="71.12" x2="375.92" y2="66.04" width="0.1524" layer="91"/>
 <wire x1="375.92" y1="66.04" x2="375.92" y2="60.96" width="0.1524" layer="91"/>
-<wire x1="375.92" y1="60.96" x2="375.92" y2="55.88" width="0.1524" layer="91"/>
-<wire x1="375.92" y1="55.88" x2="375.92" y2="53.34" width="0.1524" layer="91"/>
+<wire x1="375.92" y1="60.96" x2="375.92" y2="53.34" width="0.1524" layer="91"/>
 <wire x1="378.46" y1="76.2" x2="375.92" y2="76.2" width="0.1524" layer="91"/>
 <junction x="375.92" y="76.2"/>
@@
 <wire x1="378.46" y1="60.96" x2="375.92" y2="60.96" width="0.1524" layer="91"/>
 <junction x="375.92" y="60.96"/>
-<wire x1="378.46" y1="55.88" x2="375.92" y2="55.88" width="0.1524" layer="91"/>
-<junction x="375.92" y="55.88"/>
 </segment>
 <segment>

Commit message: added Australian Made logo, adjusted some text to make them even
Parts:
- added TP1: TPB2,54, testpad:TPB2,54
Connections:
- net 3.3V: now also TP1.TP
Other:
- note added: "3.3V"
- note added: "ACCELEROMETER"
- note added: "MAIN MICROCONTROLLER"
- note added: "TEMPERATURE"
- moved on the sheet: A, C1, C10, C2, C3, C4, C5, C6, C7, C8, C9, CLICK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
